File: OpenDeck.sch (EAGLE design)
At the start: 154 parts, among them P0 10k, P1 10k, P10 10k, P11 10k, P12 10k, P13 10k, P14 10k, P15 10k, P2 10k, P3 10k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

Commit message: potentiometer naming fixed
Parts:
- removed P0: 10k, rcl:POTENTIOMETER_PT-10
- added P16: 10k, rcl:POTENTIOMETER_PT-10
Connections:
- net GND: now also P16.1; no longer P0.1
- net MUX_1_INPUT_1: now also P1.3; no longer P0.3
- net MUX_1_INPUT_2: now also P2.3; no longer P1.3
- net MUX_1_INPUT_3: now also P3.3; no longer P2.3
- net MUX_1_INPUT_4: now also P4.3; no longer P3.3
- net MUX_1_INPUT_5: now also P5.3; no longer P4.3
- net MUX_1_INPUT_6: now also P6.3; no longer P5.3
- net MUX_1_INPUT_7: now also P7.3; no longer P6.3
- net MUX_1_INPUT_8: now also P8.3; no longer P7.3
- net MUX_2_INPUT_1: now also P9.3; no longer P8.3
- net MUX_2_INPUT_2: now also P10.3; no longer P9.3
- net MUX_2_INPUT_3: now also P11.3; no longer P10.3
- net MUX_2_INPUT_4: now also P12.3; no longer P11.3
- net MUX_2_INPUT_5: now also P13.3; no longer P12.3
- net MUX_2_INPUT_6: now also P14.3; no longer P13.3
- net MUX_2_INPUT_7: now also P15.3; no longer P14.3
- net MUX_2_INPUT_8: now also P16.3; no longer P15.3
- net VCC: now also P16.2; no longer P0.2
Other:
- moved on the sheet: P1, P10, P11, P12, P13, P14, P15, P2, P3, P4, P5, P6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
