File: bin/sch/dubfocus/ButtonsLEDs/ButtonsLEDs.brd (EAGLE design)
At the start: 143.1 x 46.1 mm, 43 parts, among them Q1 FDC6312P, Q2 FDC6312P, Q3 FDC6312P, Q4 FDC6312P, SW1 OMRON-B3W-9, SW2 OMRON-B3W-9, SW3 OMRON-B3W-9, SW4 OMRON-B3W-9, SW5 OMRON-B3W-9, SW6 OMRON-B3W-9, SW7 OMRON-B3W-9, SW8 OMRON-B3W-9, U1 74HC165, U2 74HC595-SO16

Commit message: targets: update schematics for dubfocus
Parts:
- removed CONN2, CONN4: PINHD-1X10-FFC-1MM-Z, igor_lbr:MOLEX-52271-1079
- removed Q1, Q2, Q3, Q4: FDC6312P, igor_lbr:SSOT6
- added C3, C4, C5, C6, C7, C8: 100n, igor_lbr:C0805
- added R25, R26, R27, R28, R29, R30, R31, R32, R41, R42, R43, R44, R45, R46, R47, R48, R49, R50, R51, R52, R53, R54, R55, R56, R65, R66, R67, R68, R69, R70, R71, R72, R73, R74, R75, R76, R77, R78, R79, R80, R89, R90, R91, R92, R93, R94, R95, R96: 4k7, igor_lbr:R0805
- added R33, R34, R35, R36, R37, R38, R39, R40, R57, R58, R59, R60, R61, R62, R63, R64, R81, R82, R83, R84, R85, R86, R87, R88: 750, igor_lbr:R0805
- added SW10, SW11, SW12, SW13, SW14, SW15, SW16, SW17, SW18, SW19, SW20, SW21, SW22, SW23, SW24, SW25, SW26, SW27, SW28, SW29, SW30, SW31, SW32, SW9: OMRON-B3W-9, igor_lbr:OMRON-B3W-9
- added U3, U5, U7: 74HC165, igor_lbr:SO16
- added U4, U6, U8: TPIC6B595, igor_lbr:SOIC20
- U2: value 74HC595-SO16 -> TPIC6B595; device igor_lbr:SO16 -> igor_lbr:SOIC20
- moved CONN1 326.7 mm to (432.0, 25.2), turned to 0 degrees
- moved SW8 120.0 mm to (11.5, 37.7), turned to 270 degrees
- moved R8 110.9 mm to (17.7, 40.8), flipped to the bottom
- moved R5 98.4 mm to (104.7, 40.8), flipped to the bottom
- moved SW5 87.0 mm to (98.5, 37.7), turned to 270 degrees
- moved C1 74.4 mm to (98.1, 23.5), flipped to the bottom, turned to 90 degrees
- moved U1 73.2 mm to (104.5, 25.2), flipped to the bottom, turned to 270 degrees
- moved R9 63.1 mm to (17.7, 15.7)
- moved C2 62.6 mm to (3.90, 27.1), turned to 270 degrees
- moved U2 60.0 mm to (11.6, 25.2)
- moved R24 59.5 mm to (3.10, 34.7), turned to 90 degrees
- moved R17 59.5 mm to (19.9, 15.7)
- moved R16 55.5 mm to (5.30, 34.7), turned to 270 degrees
- moved SW7 51.0 mm to (40.5, 37.7), turned to 270 degrees
- moved R4 45.9 mm to (92.3, 9.60), flipped to the bottom
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Connections:
- removed net LED1_Q: Q1.1, R17.1, U2.15
- removed net LED2_Q: Q1.3, R18.1, U2.7
- removed net LED3_Q: Q2.1, R19.1, U2.6
- removed net LED4_Q: Q2.3, R20.1, U2.5
- removed net LED5_Q: Q3.1, R21.1, U2.4
- removed net LED6_Q: Q3.3, R22.1, U2.3
- removed net LED7_Q: Q4.1, R23.1, U2.2
- removed net LED8_Q: Q4.3, R24.1, U2.1
- removed net N$1: R9.2, SW1.6-A
- removed net N$2: R10.2, SW2.6-A
- removed net N$24: Q1.6, R9.1
- removed net N$25: Q1.4, R10.1
- removed net N$26: Q2.6, R11.1
- removed net N$27: Q2.4, R12.1
- removed net N$28: Q3.6, R13.1
- removed net N$29: Q3.4, R14.1
- removed net N$3: R11.2, SW3.6-A
- removed net N$30: Q4.6, R15.1
- removed net N$31: Q4.4, R16.1
- removed net N$4: R12.2, SW4.6-A
- removed net N$5: R13.2, SW5.6-A
- removed net N$6: R15.2, SW7.6-A
- removed net N$7: R16.2, SW8.6-A
- removed net N$8: R14.2, SW6.6-A
- removed net SR_IN_DAISY_OUT: CONN1.8, U1.10
- removed net SR_OUT_DAISY_OUT: CONN1.5, U2.9
- new net BUTTON10: R26.1, SW10.1, U3.12
- new net BUTTON11: R27.1, SW11.1, U3.13
- new net BUTTON12: R28.1, SW12.1, U3.14
- new net BUTTON13: R29.1, SW13.1, U3.3
- new net BUTTON14: R30.1, SW14.1, U3.4
- new net BUTTON15: R31.1, SW15.1, U3.5
- new net BUTTON16: R32.1, SW16.1, U3.6
- new net BUTTON17: R49.1, SW17.1, U5.11
- new net BUTTON18: R50.1, SW18.1, U5.12
- new net BUTTON19: R51.1, SW19.1, U5.13
- new net BUTTON20: R52.1, SW20.1, U5.14
- new net BUTTON21: R53.1, SW21.1, U5.3
- new net BUTTON22: R54.1, SW22.1, U5.4
- new net BUTTON23: R55.1, SW23.1, U5.5
- new net BUTTON24: R56.1, SW24.1, U5.6
- new net BUTTON25: R73.1, SW25.1, U7.11
- new net BUTTON26: R74.1, SW26.1, U7.12
- new net BUTTON27: R75.1, SW27.1, U7.13
- new net BUTTON28: R76.1, SW28.1, U7.14
- new net BUTTON29: R77.1, SW29.1, U7.3
- new net BUTTON30: R78.1, SW30.1, U7.4
- new net BUTTON31: R79.1, SW31.1, U7.5
- new net BUTTON32: R80.1, SW32.1, U7.6
- new net BUTTON9: R25.1, SW9.1, U3.11
- new net LED1: R17.1, R9.2, U2.14
- new net LED10: R34.2, R42.1, U4.15
- new net LED10_R: R34.1, SW10.6-C
- new net LED11: R35.2, R43.1, U4.16
- new net LED11_R: R35.1, SW11.6-C
- new net LED12: R36.2, R44.1, U4.17
- new net LED12_R: R36.1, SW12.6-C
- new net LED13: R37.2, R45.1, U4.4
- new net LED13_R: R37.1, SW13.6-C
- new net LED14: R38.2, R46.1, U4.5
- new net LED14_R: R38.1, SW14.6-C
- new net LED15: R39.2, R47.1, U4.6
- new net LED15_R: R39.1, SW15.6-C
- new net LED16: R40.2, R48.1, U4.7
- new net LED16_R: R40.1, SW16.6-C
- new net LED17: R57.2, R65.1, U6.14
- new net LED17_R: R57.1, SW17.6-C
- new net LED18: R58.2, R66.1, U6.15
- new net LED18_R: R58.1, SW18.6-C
- new net LED19: R59.2, R67.1, U6.16
- new net LED19_R: R59.1, SW19.6-C
- new net LED1_R: R9.1, SW1.6-C
- new net LED2: R10.2, R18.1, U2.15
- new net LED20: R60.2, R68.1, U6.17
- new net LED20_R: R60.1, SW20.6-C
- new net LED21: R61.2, R69.1, U6.4
- new net LED21_R: R61.1, SW21.6-C
- new net LED22: R62.2, R70.1, U6.5
- new net LED22_R: R62.1, SW22.6-C
- new net LED23: R63.2, R71.1, U6.6
- new net LED23_R: R63.1, SW23.6-C
- new net LED24: R64.2, R72.1, U6.7
- new net LED24_R: R64.1, SW24.6-C
- new net LED25: R81.2, R89.1, U8.14
- new net LED25_R: R81.1, SW25.6-C
- new net LED26: R82.2, R90.1, U8.15
- new net LED26_R: R82.1, SW26.6-C
- new net LED27: R83.2, R91.1, U8.16
- new net LED27_R: R83.1, SW27.6-C
- new net LED28: R84.2, R92.1, U8.17
- new net LED28_R: R84.1, SW28.6-C
- new net LED29: R85.2, R93.1, U8.4
- new net LED29_R: R85.1, SW29.6-C
- new net LED2_R: R10.1, SW2.6-C
- new net LED3: R11.2, R19.1, U2.16
- new net LED30: R86.2, R94.1, U8.5
- new net LED30_R: R86.1, SW30.6-C
- new net LED31: R87.2, R95.1, U8.6
- new net LED31_R: R87.1, SW31.6-C
- new net LED32: R88.2, R96.1, U8.7
- new net LED32_R: R88.1, SW32.6-C
- new net LED3_R: R11.1, SW3.6-C
- new net LED4: R12.2, R20.1, U2.17
- new net LED4_R: R12.1, SW4.6-C
- new net LED5: R13.2, R21.1, U2.4
- new net LED5_R: R13.1, SW5.6-C
- new net LED6: R14.2, R22.1, U2.5
- new net LED6_R: R14.1, SW6.6-C
- new net LED7: R15.2, R23.1, U2.6
- new net LED7_R: R15.1, SW7.6-C
- new net LED8: R16.2, R24.1, U2.7
- new net LED8_R: R16.1, SW8.6-C
- new net LED9: R33.2, R41.1, U4.14
- new net LED9_R: R33.1, SW9.6-C
- new net SR_IN_DAISY_OUT_1: U5.9, U7.10
- new net SR_IN_DAISY_OUT_2: U3.9, U5.10
- new net SR_IN_DAISY_OUT_3: U1.9, U3.10
- new net SR_OUT_DAISY_OUT_1: U6.3, U8.18
- new net SR_OUT_DAISY_OUT_2: U4.3, U6.18
- new net SR_OUT_DAISY_OUT_3: U2.3, U4.18
- net +3V3: now also C3.1, C4.1, C5.1, C6.1, C7.1, C8.1, CONN1.2, CONN1.3, R25.2, R26.2, R27.2, R28.2, R29.2, R30.2, R31.2, R32.2, R41.2, R42.2, R43.2, R44.2, R45.2, R46.2, R47.2, R48.2, R49.2, R50.2, R51.2, R52.2, R53.2, R54.2, R55.2, R56.2, R65.2, R66.2, R67.2, R68.2, R69.2, R70.2, R71.2, R72.2, R73.2, R74.2, R75.2, R76.2, R77.2, R78.2, R79.2, R80.2, R89.2, R90.2, R91.2, R92.2, R93.2, R94.2, R95.2, R96.2, SW1.6-A, SW10.6-A, SW11.6-A, SW12.6-A, SW13.6-A, SW14.6-A, SW15.6-A, SW16.6-A, SW17.6-A, SW18.6-A, SW19.6-A, SW2.6-A, SW20.6-A, SW21.6-A, SW22.6-A, SW23.6-A, SW24.6-A, SW25.6-A, SW26.6-A, SW27.6-A, SW28.6-A, SW29.6-A, SW3.6-A, SW30.6-A, SW31.6-A, SW32.6-A, SW4.6-A, SW5.6-A, SW6.6-A, SW7.6-A, SW8.6-A, SW9.6-A, U2.2, U2.8, U3.16, U4.2, U4.8, U5.16, U6.2, U6.8, U7.16, U8.2, U8.8; no longer CONN1.10, CONN1.9, CONN2.1, CONN2.2, CONN4.2, CONN4.3, Q1.2, Q1.5, Q2.2, Q2.5, Q3.2, Q3.5, Q4.2, Q4.5, U2.10, U2.16
- net BUTTON1: now also U1.11; no longer U1.4
- net BUTTON2: now also U1.12; no longer U1.5
- net BUTTON3: now also U1.13; no longer U1.11
- net BUTTON4: now also U1.14; no longer U1.13
- net BUTTON6: now also U1.4; no longer U1.6
- net BUTTON7: now also U1.5; no longer U1.12
- net BUTTON8: now also U1.6; no longer U1.14
- net GND: now also C3.2, C4.2, C5.2, C6.2, C7.2, C8.2, SW10.3, SW11.3, SW12.3, SW13.3, SW14.3, SW15.3, SW16.3, SW17.3, SW18.3, SW19.3, SW20.3, SW21.3, SW22.3, SW23.3, SW24.3, SW25.3, SW26.3, SW27.3, SW28.3, SW29.3, SW30.3, SW31.3, SW32.3, SW9.3, U2.10, U2.11, U2.19, U3.15, U3.8, U4.10, U4.11, U4.19, U5.15, U5.8, U6.10, U6.11, U6.19, U7.15, U7.8, U8.10, U8.11, U8.19; no longer CONN2.10, CONN4.1, SW1.6-C, SW2.6-C, SW3.6-C, SW4.6-C, SW5.6-C, SW6.6-C, SW7.6-C, SW8.6-C, U2.8
- net SR_IN_CLOCK: now also CONN1.5, U3.2, U5.2, U7.2; no longer CONN1.6, CONN2.5, CONN4.4
- net SR_IN_DATA: now also CONN1.6, U7.9; no longer CONN2.3, CONN4.6, U1.9
- net SR_IN_LATCH: now also CONN1.4, U3.1, U5.1, U7.1; no longer CONN1.7, CONN2.4, CONN4.5
- net SR_OUT_CLOCK: now also CONN1.7, U2.13, U4.13, U6.13, U8.13; no longer CONN1.4, CONN2.7, CONN4.10, U2.11
- net SR_OUT_DATA: now also CONN1.9, U8.3; no longer CONN2.6, CONN4.8, U2.14
- net SR_OUT_LATCH: now also CONN1.8, U4.12, U6.12, U8.12; no longer CONN1.3, CONN2.8, CONN4.9
- net SR_OUT_OE: now also CONN1.10, U2.9, U4.9, U6.9, U8.9; no longer CONN1.2, CONN2.9, CONN4.7, U2.13
Routing:
- net +3V3: track 444.9 -> 1631.9 mm, vias 4 -> 0
- net SR_OUT_LATCH: track 114.7 -> 435.8 mm, vias 2 -> 5
- net SR_OUT_CLOCK: track 116.8 -> 433.8 mm, vias 2 -> 5
- net SR_OUT_OE: track 113.4 -> 422.7 mm, vias 2 -> 5
- net SR_IN_CLOCK: track 135.3 -> 370.9 mm, vias 3 -> 6
- net SR_IN_LATCH: track 151.7 -> 371.2 mm, vias 3 -> 5
- net SR_IN_DATA: track 168.0 -> 30.5 mm, vias 3 -> 2
- net BUTTON25: track 0.00 -> 131.0 mm
- net BUTTON17: track 0.00 -> 131.0 mm
- net BUTTON9: track 0.00 -> 131.0 mm
- net SR_OUT_DAISY_OUT_2: track 0.00 -> 130.7 mm, vias 0 -> 2
- net SR_OUT_DAISY_OUT_3: track 0.00 -> 130.2 mm, vias 0 -> 2
- net SR_IN_DAISY_OUT_1: track 0.00 -> 127.2 mm, vias 0 -> 2
- net SR_OUT_DAISY_OUT_1: track 0.00 -> 126.9 mm, vias 0 -> 2
- net SR_IN_DAISY_OUT_2: track 0.00 -> 123.4 mm, vias 0 -> 2
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Other:
- board size 143.1 x 46.1 mm -> 458.7 x 46.1 mm
- board text removed: "IN"
- board text removed: "OUT"
- board text removed: "R17/18/19/20/21/22"
