File: bin/sch/dubfocus/ButtonsLEDs/ButtonsLEDs.sch (EAGLE design)
At the start: 43 parts, among them Q1 FDC6312P, Q2 FDC6312P, Q3 FDC6312P, Q4 FDC6312P, SW1 OMRON-B3W-9, SW2 OMRON-B3W-9, SW3 OMRON-B3W-9, SW4 OMRON-B3W-9, SW5 OMRON-B3W-9, SW6 OMRON-B3W-9, SW7 OMRON-B3W-9, SW8 OMRON-B3W-9, U1 74HC165, U2 74HC595-SO16

Commit message: targets: update schematics for dubfocus
Parts:
- removed CONN2, CONN4: PINHD-1X10-FFC-1MM-Z, igor_lbr:PINHD-1X10-FFC-1MM-Z
- removed Q1, Q2, Q3, Q4: FDC6312P, igor_lbr:FDC6312P
- added C3, C4, C5, C6, C7, C8: 100n, igor_lbr:CAPACITOR-0805
- added R25, R26, R27, R28, R29, R30, R31, R32, R41, R42, R43, R44, R45, R46, R47, R48, R49, R50, R51, R52, R53, R54, R55, R56, R65, R66, R67, R68, R69, R70, R71, R72, R73, R74, R75, R76, R77, R78, R79, R80, R89, R90, R91, R92, R93, R94, R95, R96: 4k7, igor_lbr:RESISTOR-0805
- added R33, R34, R35, R36, R37, R38, R39, R40, R57, R58, R59, R60, R61, R62, R63, R64, R81, R82, R83, R84, R85, R86, R87, R88: 750, igor_lbr:RESISTOR-0805
- added SW10, SW11, SW12, SW13, SW14, SW15, SW16, SW17, SW18, SW19, SW20, SW21, SW22, SW23, SW24, SW25, SW26, SW27, SW28, SW29, SW30, SW31, SW32, SW9: OMRON-B3W-9, igor_lbr:OMRON-B3W-9
- added U3, U5, U7: 74HC165, igor_lbr:74HC165
- added U4, U6, U8: TPIC6B595, igor_lbr:TPIC6B595
- U2: value 74HC595-SO16 -> TPIC6B595; device igor_lbr:74HC595-SO16 -> igor_lbr:TPIC6B595
Connections:
- removed net LED1_Q: Q1.G1, R17.1, U2.Q0
- removed net LED2_Q: Q1.G2, R18.1, U2.Q7
- removed net LED3_Q: Q2.G1, R19.1, U2.Q6
- removed net LED4_Q: Q2.G2, R20.1, U2.Q5
- removed net LED5_Q: Q3.G1, R21.1, U2.Q4
- removed net LED6_Q: Q3.G2, R22.1, U2.Q3
- removed net LED7_Q: Q4.G1, R23.1, U2.Q2
- removed net LED8_Q: Q4.G2, R24.1, U2.Q1
- removed net N$1: R9.2, SW1-LED.A
- removed net N$2: R10.2, SW2-LED.A
- removed net N$24: Q1.D1, R9.1
- removed net N$25: Q1.D2, R10.1
- removed net N$26: Q2.D1, R11.1
- removed net N$27: Q2.D2, R12.1
- removed net N$28: Q3.D1, R13.1
- removed net N$29: Q3.D2, R14.1
- removed net N$3: R11.2, SW3-LED.A
- removed net N$30: Q4.D1, R15.1
- removed net N$31: Q4.D2, R16.1
- removed net N$4: R12.2, SW4-LED.A
- removed net N$5: R13.2, SW5-LED.A
- removed net N$6: R15.2, SW7-LED.A
- removed net N$7: R16.2, SW8-LED.A
- removed net N$8: R14.2, SW6-LED.A
- removed net SR_IN_DAISY_OUT: CONN1.8, U1.DS
- removed net SR_OUT_DAISY_OUT: CONN1.5, U2.Q7S
- new net BUTTON10: R26.1, SW10-SW.1, U3.D1
- new net BUTTON11: R27.1, SW11-SW.1, U3.D2
- new net BUTTON12: R28.1, SW12-SW.1, U3.D3
- new net BUTTON13: R29.1, SW13-SW.1, U3.D4
- new net BUTTON14: R30.1, SW14-SW.1, U3.D5
- new net BUTTON15: R31.1, SW15-SW.1, U3.D6
- new net BUTTON16: R32.1, SW16-SW.1, U3.D7
- new net BUTTON17: R49.1, SW17-SW.1, U5.D0
- new net BUTTON18: R50.1, SW18-SW.1, U5.D1
- new net BUTTON19: R51.1, SW19-SW.1, U5.D2
- new net BUTTON20: R52.1, SW20-SW.1, U5.D3
- new net BUTTON21: R53.1, SW21-SW.1, U5.D4
- new net BUTTON22: R54.1, SW22-SW.1, U5.D5
- new net BUTTON23: R55.1, SW23-SW.1, U5.D6
- new net BUTTON24: R56.1, SW24-SW.1, U5.D7
- new net BUTTON25: R73.1, SW25-SW.1, U7.D0
- new net BUTTON26: R74.1, SW26-SW.1, U7.D1
- new net BUTTON27: R75.1, SW27-SW.1, U7.D2
- new net BUTTON28: R76.1, SW28-SW.1, U7.D3
- new net BUTTON29: R77.1, SW29-SW.1, U7.D4
- new net BUTTON30: R78.1, SW30-SW.1, U7.D5
- new net BUTTON31: R79.1, SW31-SW.1, U7.D6
- new net BUTTON32: R80.1, SW32-SW.1, U7.D7
- new net BUTTON9: R25.1, SW9-SW.1, U3.D0
- new net LED1: R17.1, R9.2, U2.D4
- new net LED10: R34.2, R42.1, U4.D5
- new net LED10_R: R34.1, SW10-LED.C
- new net LED11: R35.2, R43.1, U4.D6
- new net LED11_R: R35.1, SW11-LED.C
- new net LED12: R36.2, R44.1, U4.D7
- new net LED12_R: R36.1, SW12-LED.C
- new net LED13: R37.2, R45.1, U4.D0
- new net LED13_R: R37.1, SW13-LED.C
- new net LED14: R38.2, R46.1, U4.D1
- new net LED14_R: R38.1, SW14-LED.C
- new net LED15: R39.2, R47.1, U4.D2
- new net LED15_R: R39.1, SW15-LED.C
- new net LED16: R40.2, R48.1, U4.D3
- new net LED16_R: R40.1, SW16-LED.C
- new net LED17: R57.2, R65.1, U6.D4
- new net LED17_R: R57.1, SW17-LED.C
- new net LED18: R58.2, R66.1, U6.D5
- new net LED18_R: R58.1, SW18-LED.C
- new net LED19: R59.2, R67.1, U6.D6
- new net LED19_R: R59.1, SW19-LED.C
- new net LED1_R: R9.1, SW1-LED.C
- new net LED2: R10.2, R18.1, U2.D5
- new net LED20: R60.2, R68.1, U6.D7
- new net LED20_R: R60.1, SW20-LED.C
- new net LED21: R61.2, R69.1, U6.D0
- new net LED21_R: R61.1, SW21-LED.C
- new net LED22: R62.2, R70.1, U6.D1
- new net LED22_R: R62.1, SW22-LED.C
- new net LED23: R63.2, R71.1, U6.D2
- new net LED23_R: R63.1, SW23-LED.C
- new net LED24: R64.2, R72.1, U6.D3
- new net LED24_R: R64.1, SW24-LED.C
- new net LED25: R81.2, R89.1, U8.D4
- new net LED25_R: R81.1, SW25-LED.C
- new net LED26: R82.2, R90.1, U8.D5
- new net LED26_R: R82.1, SW26-LED.C
- new net LED27: R83.2, R91.1, U8.D6
- new net LED27_R: R83.1, SW27-LED.C
- new net LED28: R84.2, R92.1, U8.D7
- new net LED28_R: R84.1, SW28-LED.C
- new net LED29: R85.2, R93.1, U8.D0
- new net LED29_R: R85.1, SW29-LED.C
- new net LED2_R: R10.1, SW2-LED.C
- new net LED3: R11.2, R19.1, U2.D6
- new net LED30: R86.2, R94.1, U8.D1
- new net LED30_R: R86.1, SW30-LED.C
- new net LED31: R87.2, R95.1, U8.D2
- new net LED31_R: R87.1, SW31-LED.C
- new net LED32: R88.2, R96.1, U8.D3
- new net LED32_R: R88.1, SW32-LED.C
- new net LED3_R: R11.1, SW3-LED.C
- new net LED4: R12.2, R20.1, U2.D7
- new net LED4_R: R12.1, SW4-LED.C
- new net LED5: R13.2, R21.1, U2.D0
- new net LED5_R: R13.1, SW5-LED.C
- new net LED6: R14.2, R22.1, U2.D1
- new net LED6_R: R14.1, SW6-LED.C
- new net LED7: R15.2, R23.1, U2.D2
- new net LED7_R: R15.1, SW7-LED.C
- new net LED8: R16.2, R24.1, U2.D3
- new net LED8_R: R16.1, SW8-LED.C
- new net LED9: R33.2, R41.1, U4.D4
- new net LED9_R: R33.1, SW9-LED.C
- new net SR_IN_DAISY_OUT_1: U5.Q7, U7.DS
- new net SR_IN_DAISY_OUT_2: U3.Q7, U5.DS
- new net SR_IN_DAISY_OUT_3: U1.Q7, U3.DS
- new net SR_OUT_DAISY_OUT_1: U6.SER_IN, U8.SER_OUT
- new net SR_OUT_DAISY_OUT_2: U4.SER_IN, U6.SER_OUT
- new net SR_OUT_DAISY_OUT_3: U2.SER_IN, U4.SER_OUT
- net +3V3: now also C3.1, C4.1, C5.1, C6.1, C7.1, C8.1, CONN1.2, CONN1.3, R25.2, R26.2, R27.2, R28.2, R29.2, R30.2, R31.2, R32.2, R41.2, R42.2, R43.2, R44.2, R45.2, R46.2, R47.2, R48.2, R49.2, R50.2, R51.2, R52.2, R53.2, R54.2, R55.2, R56.2, R65.2, R66.2, R67.2, R68.2, R69.2, R70.2, R71.2, R72.2, R73.2, R74.2, R75.2, R76.2, R77.2, R78.2, R79.2, R80.2, R89.2, R90.2, R91.2, R92.2, R93.2, R94.2, R95.2, R96.2, SW1-LED.A, SW10-LED.A, SW11-LED.A, SW12-LED.A, SW13-LED.A, SW14-LED.A, SW15-LED.A, SW16-LED.A, SW17-LED.A, SW18-LED.A, SW19-LED.A, SW2-LED.A, SW20-LED.A, SW21-LED.A, SW22-LED.A, SW23-LED.A, SW24-LED.A, SW25-LED.A, SW26-LED.A, SW27-LED.A, SW28-LED.A, SW29-LED.A, SW3-LED.A, SW30-LED.A, SW31-LED.A, SW32-LED.A, SW4-LED.A, SW5-LED.A, SW6-LED.A, SW7-LED.A, SW8-LED.A, SW9-LED.A, U2.!SRCLR, U3.VCC, U4.!SRCLR, U4.VCC, U5.VCC, U6.!SRCLR, U6.VCC, U7.VCC, U8.!SRCLR, U8.VCC; no longer CONN1.10, CONN1.9, CONN2.1, CONN2.2, CONN4.2, CONN4.3, Q1.S1, Q1.S2, Q2.S1, Q2.S2, Q3.S1, Q3.S2, Q4.S1, Q4.S2, U2.!MR
- net BUTTON1: now also U1.D0; no longer U1.D5
- net BUTTON2: now also U1.D1; no longer U1.D6
- net BUTTON3: now also U1.D2; no longer U1.D0
- net BUTTON4: now also U1.D3; no longer U1.D2
- net BUTTON6: now also U1.D5; no longer U1.D7
- net BUTTON7: now also U1.D6; no longer U1.D1
- net BUTTON8: now also U1.D7; no longer U1.D3
- net GND: now also C3.2, C4.2, C5.2, C6.2, C7.2, C8.2, SW10-SW.2, SW11-SW.2, SW12-SW.2, SW13-SW.2, SW14-SW.2, SW15-SW.2, SW16-SW.2, SW17-SW.2, SW18-SW.2, SW19-SW.2, SW20-SW.2, SW21-SW.2, SW22-SW.2, SW23-SW.2, SW24-SW.2, SW25-SW.2, SW26-SW.2, SW27-SW.2, SW28-SW.2, SW29-SW.2, SW30-SW.2, SW31-SW.2, SW32-SW.2, SW9-SW.2, U2.GND@10, U2.GND@11, U2.GND@19, U3.!CE, U3.GND, U4.GND@10, U4.GND@11, U4.GND@19, U5.!CE, U5.GND, U6.GND@10, U6.GND@11, U6.GND@19, U7.!CE, U7.GND, U8.GND@10, U8.GND@11, U8.GND@19; no longer CONN2.10, CONN4.1, SW1-LED.C, SW2-LED.C, SW3-LED.C, SW4-LED.C, SW5-LED.C, SW6-LED.C, SW7-LED.C, SW8-LED.C, U2.GND
- net SR_IN_CLOCK: now also CONN1.5, U3.CP, U5.CP, U7.CP; no longer CONN1.6, CONN2.5, CONN4.4
- net SR_IN_DATA: now also CONN1.6, U7.Q7; no longer CONN2.3, CONN4.6, U1.Q7
- net SR_IN_LATCH: now also CONN1.4, U3.!PL, U5.!PL, U7.!PL; no longer CONN1.7, CONN2.4, CONN4.5
- net SR_OUT_CLOCK: now also CONN1.7, U2.SRCK, U4.SRCK, U6.SRCK, U8.SRCK; no longer CONN1.4, CONN2.7, CONN4.10, U2.SHCP
- net SR_OUT_DATA: now also CONN1.9, U8.SER_IN; no longer CONN2.6, CONN4.8, U2.DS
- net SR_OUT_LATCH: now also CONN1.8, U2.RCK, U4.RCK, U6.RCK, U8.RCK; no longer CONN1.3, CONN2.8, CONN4.9, U2.STCP
- net SR_OUT_OE: now also CONN1.10, U2.!G/OE, U4.!G/OE, U6.!G/OE, U8.!G/OE; no longer CONN1.2, CONN2.9, CONN4.7, U2.!OE
Other:
- note removed: "Note: same-sided flat cables should be used, such as Molex 15267-0257"
- moved on the sheet: C1, C2, CONN1, R1, R10, R11, R12, R13, R14, R15, R16, R17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
