File: bin/sch/dubfocus/MBO/MBO.brd (EAGLE design)
At the start: 72 x 77 mm, 32 parts, among them U1 STM32F405RGT6-10X10-HS, U2 MC14067BDWR2G-SO24W, Y1 16MHz

Commit message: targets: update schematics for dubfocus
Parts:
- removed C1, C20: 2.2u, igor_lbr:C0805
- removed C17, C2, C3, C4, C5, C6, C7: 100n, igor_lbr:C0805
- removed C21: 1u, igor_lbr:C0805
- removed C8, C9: 22p, igor_lbr:C0805
- removed CONN19: PINHD-1X05-JST-XH-H, igor_lbr:JST-XH-05P-H
- removed CONN8: PINHD-1X20-SMD, igor_lbr:MOLEX-52271-2079
- removed CONN9: PINHD-1X05-TH-2.54MM, igor_lbr:1X05-2.54
- removed L1: FERRITE_BEAD-BLM21PG221SN1D, igor_lbr:L0805
- removed R40, R41: 22, igor_lbr:R0805
- removed Y1: 16MHz, igor_lbr:HC49US
- added FADER1, FADER10, FADER11, FADER12, FADER13, FADER14, FADER15, FADER16, FADER2, FADER3, FADER4, FADER5, FADER6, FADER7, FADER8, FADER9: RS6011P, igor_lbr:RS6011*P
- added SW1: (no value), igor_lbr:TACT_SW_6X6MM
- R1: value 510 -> 0
- U1: value STM32F405RGT6-10X10-HS -> STM32F411-BLACK_PILL; device igor_lbr:TQFP-64-10X10-HS -> igor_lbr:STM32F411-BLACK_PILL
- moved CONN1 412.2 mm to (426.5, 54.8), flipped to the bottom
- moved R2 408.3 mm to (415.9, 57.4), flipped to the bottom, turned to 90 degrees
- moved U2 382.3 mm to (426.5, 21.5), flipped to the bottom, turned to 270 degrees
- moved R1 376.6 mm to (409.7, 17.9), flipped to the bottom, turned to 180 degrees
- moved C12 373.2 mm to (419.3, 13.2), flipped to the bottom, turned to 270 degrees
- moved C18 371.7 mm to (407.7, 72.2), flipped to the bottom, turned to 90 degrees
- moved C19 368.4 mm to (405.1, 68.8), flipped to the bottom, turned to 180 degrees
- moved VR1 368.2 mm to (411.6, 66.6), flipped to the bottom, turned to 0 degrees
- moved C10 368.1 mm to (417.2, 68.0), flipped to the bottom, turned to 270 degrees
- moved C11 366.8 mm to (417.2, 63.6), flipped to the bottom
- moved U1 366.7 mm to (397.5, 39.5), flipped to the bottom, turned to 0 degrees
- moved CONN2 366.2 mm to (426.5, 39.8), flipped to the bottom
- moved R3 364.1 mm to (387.0, 21.4), flipped to the bottom, turned to 270 degrees
Connections:
- removed net BOOT0: R1.1, U1.60
- removed net N$16: C1.1, U1.31
- removed net N$17: C20.2, U1.47
- removed net NRST: C17.1, CONN9.5, U1.7
- removed net OSC_IN: C8.2, U1.6, Y1.1
- removed net OSC_OUT: C9.2, U1.5, Y1.2
- removed net SWDCLK: CONN9.2, U1.49
- removed net SWDIO: CONN9.4, U1.46
- removed net USB_DM: R41.1, U1.44
- removed net USB_DM-R: CONN19.3, R41.2
- removed net USB_DP: R40.1, U1.45
- removed net USB_DP-R: CONN19.2, R40.2
- net +3V3: now also FADER1.3, FADER10.3, FADER11.3, FADER12.3, FADER13.3, FADER14.3, FADER15.3, FADER16.3, FADER2.3, FADER3.3, FADER4.3, FADER5.3, FADER6.3, FADER7.3, FADER8.3, FADER9.3; no longer C2.1, C21.1, C3.1, C4.1, C5.1, C6.1, C7.1, CONN8.1, CONN8.2, CONN9.1, U1.1, U1.13, U1.19, U1.32, U1.48, U1.64
- net +5V: now also U1.P2.1; no longer CONN19.1
- net AGND: now also FADER1.1, FADER1.S1, FADER1.S2, FADER1.S3, FADER1.S4, FADER1.S5, FADER10.1, FADER10.S1, FADER10.S2, FADER10.S3, FADER10.S4, FADER10.S5, FADER11.1, FADER11.S1, FADER11.S2, FADER11.S3, FADER11.S4, FADER11.S5, FADER12.1, FADER12.S1, FADER12.S2, FADER12.S3, FADER12.S4, FADER12.S5, FADER13.1, FADER13.S1, FADER13.S2, FADER13.S3, FADER13.S4, FADER13.S5, FADER14.1, FADER14.S1, FADER14.S2, FADER14.S3, FADER14.S4, FADER14.S5, FADER15.1, FADER15.S1, FADER15.S2, FADER15.S3, FADER15.S4, FADER15.S5, FADER16.1, FADER16.S1, FADER16.S2, FADER16.S3, FADER16.S4, FADER16.S5, FADER2.1, FADER2.S1, FADER2.S2, FADER2.S3, FADER2.S4, FADER2.S5, FADER3.1, FADER3.S1, FADER3.S2, FADER3.S3, FADER3.S4, FADER3.S5, FADER4.1, FADER4.S1, FADER4.S2, FADER4.S3, FADER4.S4, FADER4.S5, FADER5.1, FADER5.S1, FADER5.S2, FADER5.S3, FADER5.S4, FADER5.S5, FADER6.1, FADER6.S1, FADER6.S2, FADER6.S3, FADER6.S4, FADER6.S5, FADER7.1, FADER7.S1, FADER7.S2, FADER7.S3, FADER7.S4, FADER7.S5, FADER8.1, FADER8.S1, FADER8.S2, FADER8.S3, FADER8.S4, FADER8.S5, FADER9.1, FADER9.S1, FADER9.S2, FADER9.S3, FADER9.S4, FADER9.S5, R1.2; no longer C21.2, C7.2, CONN8.3, CONN8.4, L1.2, U1.12
- net BTLDR_BUTTON: now also SW1.A1, U1.P2.18; no longer CONN19.4, U1.54
- net FADER1: now also FADER1.2, U2.2; no longer CONN8.5, U2.6
- net FADER10: now also FADER10.2; no longer CONN8.15
- net FADER11: now also FADER11.2; no longer CONN8.14
- net FADER12: now also FADER12.2; no longer CONN8.13
- net FADER13: now also FADER13.2; no longer CONN8.12
- net FADER14: now also FADER14.2; no longer CONN8.11
- net FADER15: now also FADER15.2; no longer CONN8.10
- net FADER16: now also FADER16.2; no longer CONN8.9
- net FADER2: now also FADER2.2, U2.3; no longer CONN8.6, U2.7
- net FADER3: now also FADER3.2, U2.4; no longer CONN8.7, U2.8
- net FADER4: now also FADER4.2, U2.5; no longer CONN8.8, U2.9
- net FADER5: now also FADER5.2, U2.6; no longer CONN8.17, U2.5
- net FADER6: now also FADER6.2, U2.7; no longer CONN8.18, U2.4
- net FADER7: now also FADER7.2, U2.8; no longer CONN8.19, U2.3
- net FADER8: now also FADER8.2, U2.9; no longer CONN8.20, U2.2
- net FADER9: now also FADER9.2; no longer CONN8.16
- net GND: now also R1.1, SW1.B1, U1.P1.19, U1.P2.2; no longer C1.2, C17.2, C2.2, C20.1, C3.2, C4.2, C5.2, C6.2, C8.1, C9.1, CONN19.5, CONN9.3, L1.1, R1.2, U1.18, U1.63
- net MUX_COMMON_1: now also CONN2.10, U1.P2.13; no longer CONN2.7, U1.23
- net MUX_COMMON_2: now also CONN2.9, U1.P2.12; no longer CONN2.8, U1.22
- net MUX_COMMON_3: now also CONN2.8, U1.P2.11; no longer CONN2.9, U1.21
- net MUX_COMMON_4: now also CONN2.7, U1.P2.10; no longer CONN2.10, U1.20
- net MUX_COMMON_5: now also U1.P2.14; no longer U1.15
- net MUX_S0: now also U1.P2.8; no longer U1.57
- net MUX_S1: now also U1.P1.7; no longer U1.58
- net MUX_S2: now also U1.P2.9; no longer U1.56
- net MUX_S3: now also U1.P1.10; no longer U1.55
- net SR_IN_CLOCK: now also CONN1.6, U1.P2.5; no longer CONN1.7, U1.36
- net SR_IN_DATA: now also U1.P1.4; no longer U1.34
- net SR_IN_LATCH: now also CONN1.7, U1.P2.6; no longer CONN1.6, U1.35
- net SR_OUT_CLOCK: now also CONN1.4, U1.P2.4; no longer CONN1.1, U1.26
- net SR_OUT_DATA: now also CONN1.2, U1.P1.2; no longer CONN1.3, U1.28
- net SR_OUT_LATCH: now also CONN1.3, U1.P1.3; no longer CONN1.2, U1.27
- net SR_OUT_OE: now also CONN1.1, U1.P1.1; no longer CONN1.4, U1.29
Routing:
- net FADER1: track 72.3 -> 436.8 mm
- net FADER2: track 70.1 -> 408.8 mm
- net FADER3: track 67.4 -> 380.9 mm
- net FADER5: track 33.5 -> 326.2 mm
- net FADER4: track 64.9 -> 354.2 mm
- net +3V3: track 304.3 -> 593.3 mm
- net FADER6: track 32.3 -> 298.3 mm
- net FADER7: track 31.0 -> 270.6 mm
- net FADER8: track 25.9 -> 242.4 mm
- net FADER9: track 33.3 -> 197.4 mm
- net BTLDR_BUTTON: track 27.5 -> 174.5 mm
- net FADER10: track 35.0 -> 169.9 mm
- net FADER11: track 36.3 -> 141.7 mm
- net FADER12: track 37.4 -> 113.7 mm
- net AGND: track 6.47 -> 73.3 mm, vias 12 -> 8
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- removed copper zone on layer 1, net AGND
- removed copper zone on layer 16, net GND
Other:
- board size 72 x 77 mm -> 447 x 78 mm
- board text added: "BTLDR"
- board text removed: "FADERS"
