File: bin/sch/dubfocus/MBO/MBO.sch (EAGLE design)
At the start: 32 parts, among them U1 STM32F405RGT6-10X10-HS, U2 MC14067BDWR2G-SO24W, Y1 16MHz

Commit message: targets: update schematics for dubfocus
Parts:
- removed C1, C20: 2.2u, igor_lbr:CAPACITOR-0805
- removed C17, C2, C3, C4, C5, C6, C7: 100n, igor_lbr:CAPACITOR-0805
- removed C21: 1u, igor_lbr:CAPACITOR-0805
- removed C8, C9: 22p, igor_lbr:CAPACITOR-0805
- removed CONN19: PINHD-1X05-JST-XH-H, igor_lbr:PINHD-1X05-JST-XH-H
- removed CONN8: PINHD-1X20-SMD, igor_lbr:PINHD-1X20-SMD
- removed CONN9: PINHD-1X05-TH-2.54MM, igor_lbr:PINHD-1X05-TH-2.54MM
- removed L1: FERRITE_BEAD-BLM21PG221SN1D, igor_lbr:FERRITE_BEAD-BLM21PG221SN1D
- removed R40, R41: 22, igor_lbr:RESISTOR-0805
- removed Y1: 16MHz, igor_lbr:CRYSTAL-HC49
- added FADER1, FADER10, FADER11, FADER12, FADER13, FADER14, FADER15, FADER16, FADER2, FADER3, FADER4, FADER5, FADER6, FADER7, FADER8, FADER9: RS6011P, igor_lbr:RS6011P
- added SW1: (no value), igor_lbr:SWITCH-TACT-TH-6X6MM
- R1: value 510 -> 0
- U1: value STM32F405RGT6-10X10-HS -> STM32F411-BLACK_PILL; device igor_lbr:STM32F405RGT6-10X10-HS -> igor_lbr:STM32F411-BLACK_PILL
Connections:
- removed net BOOT0: R1.1, U1.BOOT0
- removed net N$16: C1.1, U1.VCAP
- removed net N$17: C20.2, U1.VCAP@2
- removed net NRST: C17.1, CONN9.5, U1.NRST
- removed net OSC_IN: C8.2, U1.PH1, Y1.1
- removed net OSC_OUT: C9.2, U1.PH0, Y1.2
- removed net SWDCLK: CONN9.2, U1.PA14
- removed net SWDIO: CONN9.4, U1.PA13
- removed net USB_DM: R41.1, U1.PA11
- removed net USB_DM-R: CONN19.3, R41.2
- removed net USB_DP: R40.1, U1.PA12
- removed net USB_DP-R: CONN19.2, R40.2
- net +3V3: now also FADER1-POT.3, FADER10-POT.3, FADER11-POT.3, FADER12-POT.3, FADER13-POT.3, FADER14-POT.3, FADER15-POT.3, FADER16-POT.3, FADER2-POT.3, FADER3-POT.3, FADER4-POT.3, FADER5-POT.3, FADER6-POT.3, FADER7-POT.3, FADER8-POT.3, FADER9-POT.3; no longer C2.1, C21.1, C3.1, C4.1, C5.1, C6.1, C7.1, CONN8.1, CONN8.2, CONN9.1, U1.VBAT, U1.VDD, U1.VDD@1, U1.VDD@2, U1.VDD@4, U1.VDDA
- net +5V: now also U1.+5V@1; no longer CONN19.1
- net AGND: now also FADER1-POT.1, FADER1-S1.S, FADER1-S2.S, FADER1-S3.S, FADER1-S4.S, FADER1-S5.S, FADER10-POT.1, FADER10-S1.S, FADER10-S2.S, FADER10-S3.S, FADER10-S4.S, FADER10-S5.S, FADER11-POT.1, FADER11-S1.S, FADER11-S2.S, FADER11-S3.S, FADER11-S4.S, FADER11-S5.S, FADER12-POT.1, FADER12-S1.S, FADER12-S2.S, FADER12-S3.S, FADER12-S4.S, FADER12-S5.S, FADER13-POT.1, FADER13-S1.S, FADER13-S2.S, FADER13-S3.S, FADER13-S4.S, FADER13-S5.S, FADER14-POT.1, FADER14-S1.S, FADER14-S2.S, FADER14-S3.S, FADER14-S4.S, FADER14-S5.S, FADER15-POT.1, FADER15-S1.S, FADER15-S2.S, FADER15-S3.S, FADER15-S4.S, FADER15-S5.S, FADER16-POT.1, FADER16-S1.S, FADER16-S2.S, FADER16-S3.S, FADER16-S4.S, FADER16-S5.S, FADER2-POT.1, FADER2-S1.S, FADER2-S2.S, FADER2-S3.S, FADER2-S4.S, FADER2-S5.S, FADER3-POT.1, FADER3-S1.S, FADER3-S2.S, FADER3-S3.S, FADER3-S4.S, FADER3-S5.S, FADER4-POT.1, FADER4-S1.S, FADER4-S2.S, FADER4-S3.S, FADER4-S4.S, FADER4-S5.S, FADER5-POT.1, FADER5-S1.S, FADER5-S2.S, FADER5-S3.S, FADER5-S4.S, FADER5-S5.S, FADER6-POT.1, FADER6-S1.S, FADER6-S2.S, FADER6-S3.S, FADER6-S4.S, FADER6-S5.S, FADER7-POT.1, FADER7-S1.S, FADER7-S2.S, FADER7-S3.S, FADER7-S4.S, FADER7-S5.S, FADER8-POT.1, FADER8-S1.S, FADER8-S2.S, FADER8-S3.S, FADER8-S4.S, FADER8-S5.S, FADER9-POT.1, FADER9-S1.S, FADER9-S2.S, FADER9-S3.S, FADER9-S4.S, FADER9-S5.S, R1.2; no longer C21.2, C7.2, CONN8.3, CONN8.4, L1.2, U1.VSSA
- net BTLDR_BUTTON: now also SW1.1, U1.C14; no longer CONN19.4, U1.PD2
- net FADER1: now also FADER1-POT.2, U2.Y7; no longer CONN8.5, U2.Y3
- net FADER10: now also FADER10-POT.2; no longer CONN8.15
- net FADER11: now also FADER11-POT.2; no longer CONN8.14
- net FADER12: now also FADER12-POT.2; no longer CONN8.13
- net FADER13: now also FADER13-POT.2; no longer CONN8.12
- net FADER14: now also FADER14-POT.2; no longer CONN8.11
- net FADER15: now also FADER15-POT.2; no longer CONN8.10
- net FADER16: now also FADER16-POT.2; no longer CONN8.9
- net FADER2: now also FADER2-POT.2, U2.Y6; no longer CONN8.6, U2.Y2
- net FADER3: now also FADER3-POT.2, U2.Y5; no longer CONN8.7, U2.Y1
- net FADER4: now also FADER4-POT.2, U2.Y4; no longer CONN8.8, U2.Y0
- net FADER5: now also FADER5-POT.2, U2.Y3; no longer CONN8.17, U2.Y4
- net FADER6: now also FADER6-POT.2, U2.Y2; no longer CONN8.18, U2.Y5
- net FADER7: now also FADER7-POT.2, U2.Y1; no longer CONN8.19, U2.Y6
- net FADER8: now also FADER8-POT.2, U2.Y0; no longer CONN8.20, U2.Y7
- net FADER9: now also FADER9-POT.2; no longer CONN8.16
- net GND: now also R1.1, SW1.2, U1.GND, U1.GND@1; no longer C1.2, C17.2, C2.2, C20.1, C3.2, C4.2, C5.2, C6.2, C8.1, C9.1, CONN19.5, CONN9.3, L1.1, R1.2, U1.VSS, U1.VSS@1
- net MUX_COMMON_1: now also CONN2.10, U1.A2; no longer CONN2.7, U1.PA7
- net MUX_COMMON_2: now also CONN2.9, U1.A3; no longer CONN2.8, U1.PA6
- net MUX_COMMON_3: now also CONN2.8, U1.A4; no longer CONN2.9, U1.PA5
- net MUX_COMMON_4: now also CONN2.7, U1.A5; no longer CONN2.10, U1.PA4
- net MUX_COMMON_5: now also U1.A1; no longer U1.PA1
- net MUX_S0: now also U1.A7; no longer U1.PB5
- net MUX_S1: now also U1.A10; no longer U1.PB6
- net MUX_S2: now also U1.A6; no longer U1.PB4
- net MUX_S3: now also U1.A15; no longer U1.PB3
- net SR_IN_CLOCK: now also CONN1.6, U1.B2; no longer CONN1.7, U1.PB15
- net SR_IN_DATA: now also U1.B15; no longer U1.PB13
- net SR_IN_LATCH: now also CONN1.7, U1.B1; no longer CONN1.6, U1.PB14
- net SR_OUT_CLOCK: now also CONN1.4, U1.B10; no longer CONN1.1, U1.PB0
- net SR_OUT_DATA: now also CONN1.2, U1.B13; no longer CONN1.3, U1.PB2
- net SR_OUT_LATCH: now also CONN1.3, U1.B14; no longer CONN1.2, U1.PB1
- net SR_OUT_OE: now also CONN1.1, U1.B12; no longer CONN1.4, U1.PB10
Other:
- note removed: "VBAT"
- note removed: "VDD/19"
- note removed: "VDD/32"
- note removed: "VDD/48"
- note removed: "VDD/64"
- note removed: "VDDA"
- moved on the sheet: C10, C11, C12, C18, C19, CONN1, CONN2, R1, R2, R3, U2, VR1
