File: bin/sch/dubfocus/Pots/Pots.brd (EAGLE design)
At the start: 135.2 x 99.8 mm, 27 parts, among them U1 MC14067BDWR2G-SO24W

Commit message: targets: update schematics for dubfocus
Parts:
- removed CONN2, CONN3: PINHD-1X10-FFC-1MM-Z, igor_lbr:MOLEX-52271-1079
- added C4, C5, C6: 100n, igor_lbr:C0805
- added R21, R22, R23, R24, R25, R26, R27, R28, R29, R30, R31, R32, R33, R34, R35, R36, R37, R38, R39, R40, R41, R42, R43, R44, R45, R46, R47, R48, R49, R50, R51, R52, R53, R54, R55, R56, R57, R58, R59, R60, R61, R62, R63, R64: 10k, igor_lbr:PTV09A-4025F-B103
- added U2, U3, U4: MC14067BDWR2G-SO24W, igor_lbr:SO24-W
- R17, R18, R19, R20: value 0 -> 10k; device igor_lbr:R0805 -> igor_lbr:PTV09A-4025F-B103
- moved CONN1 360.3 mm to (427.8, 23.7)
- moved C2 354.6 mm to (426.9, 30.0)
- moved C1 353.6 mm to (426.8, 33.6), turned to 0 degrees
- moved R17 90.2 mm to (123.3, 86.2), flipped to the top
- moved R18 76.4 mm to (123.3, 61.2), flipped to the top
- moved R19 67.6 mm to (123.3, 36.2), flipped to the top
- moved R20 65.9 mm to (123.3, 11.2), flipped to the top
- moved R13 33.3 mm to (94.3, 86.2)
- moved R14 33.3 mm to (94.3, 61.2)
- moved R15 33.3 mm to (94.3, 36.2)
- moved R16 33.3 mm to (94.3, 11.2)
- moved R10 22.3 mm to (65.3, 61.2)
- moved R11 22.3 mm to (65.3, 36.2)
- moved R12 22.3 mm to (65.3, 11.2)
- moved R9 22.3 mm to (65.3, 86.2)
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Connections:
- removed net MUX_COMMON: R17.1, R18.1, R19.1, R20.1, U1.1
- new net POT17: R17.2, U2.21
- new net POT18: R18.2, U2.20
- new net POT19: R19.2, U2.19
- new net POT20: R20.2, U2.18
- new net POT21: R21.2, U2.23
- new net POT22: R22.2, U2.22
- new net POT23: R23.2, U2.17
- new net POT24: R24.2, U2.16
- new net POT25: R25.2, U2.2
- new net POT26: R26.2, U2.3
- new net POT27: R27.2, U2.8
- new net POT28: R28.2, U2.9
- new net POT29: R29.2, U2.4
- new net POT30: R30.2, U2.5
- new net POT31: R31.2, U2.6
- new net POT32: R32.2, U2.7
- new net POT33: R33.2, U3.21
- new net POT34: R34.2, U3.20
- new net POT35: R35.2, U3.19
- new net POT36: R36.2, U3.18
- new net POT37: R37.2, U3.23
- new net POT38: R38.2, U3.22
- new net POT39: R39.2, U3.17
- new net POT40: R40.2, U3.16
- new net POT41: R41.2, U3.2
- new net POT42: R42.2, U3.3
- new net POT43: R43.2, U3.8
- new net POT44: R44.2, U3.9
- new net POT45: R45.2, U3.4
- new net POT46: R46.2, U3.5
- new net POT47: R47.2, U3.6
- new net POT48: R48.2, U3.7
- new net POT49: R49.2, U4.21
- new net POT50: R50.2, U4.20
- new net POT51: R51.2, U4.19
- new net POT52: R52.2, U4.18
- new net POT53: R53.2, U4.23
- new net POT54: R54.2, U4.22
- new net POT55: R55.2, U4.17
- new net POT56: R56.2, U4.16
- new net POT57: R57.2, U4.2
- new net POT58: R58.2, U4.3
- new net POT59: R59.2, U4.8
- new net POT60: R60.2, U4.9
- new net POT61: R61.2, U4.4
- new net POT62: R62.2, U4.5
- new net POT63: R63.2, U4.6
- new net POT64: R64.2, U4.7
- net +3V3: now also C4.2, C5.2, C6.2, R17.3, R18.3, R19.3, R20.3, R21.3, R22.3, R23.3, R24.3, R25.3, R26.3, R27.3, R28.3, R29.3, R30.3, R31.3, R32.3, R33.3, R34.3, R35.3, R36.3, R37.3, R38.3, R39.3, R40.3, R41.3, R42.3, R43.3, R44.3, R45.3, R46.3, R47.3, R48.3, R49.3, R50.3, R51.3, R52.3, R53.3, R54.3, R55.3, R56.3, R57.3, R58.3, R59.3, R60.3, R61.3, R62.3, R63.3, R64.3, U2.24, U3.24, U4.24; no longer CONN2.6, CONN3.5
- net GND: now also C4.1, C5.1, C6.1, R17.1, R17.S1, R17.S2, R18.1, R18.S1, R18.S2, R19.1, R19.S1, R19.S2, R20.1, R20.S1, R20.S2, R21.1, R21.S1, R21.S2, R22.1, R22.S1, R22.S2, R23.1, R23.S1, R23.S2, R24.1, R24.S1, R24.S2, R25.1, R25.S1, R25.S2, R26.1, R26.S1, R26.S2, R27.1, R27.S1, R27.S2, R28.1, R28.S1, R28.S2, R29.1, R29.S1, R29.S2, R30.1, R30.S1, R30.S2, R31.1, R31.S1, R31.S2, R32.1, R32.S1, R32.S2, R33.1, R33.S1, R33.S2, R34.1, R34.S1, R34.S2, R35.1, R35.S1, R35.S2, R36.1, R36.S1, R36.S2, R37.1, R37.S1, R37.S2, R38.1, R38.S1, R38.S2, R39.1, R39.S1, R39.S2, R40.1, R40.S1, R40.S2, R41.1, R41.S1, R41.S2, R42.1, R42.S1, R42.S2, R43.1, R43.S1, R43.S2, R44.1, R44.S1, R44.S2, R45.1, R45.S1, R45.S2, R46.1, R46.S1, R46.S2, R47.1, R47.S1, R47.S2, R48.1, R48.S1, R48.S2, R49.1, R49.S1, R49.S2, R50.1, R50.S1, R50.S2, R51.1, R51.S1, R51.S2, R52.1, R52.S1, R52.S2, R53.1, R53.S1, R53.S2, R54.1, R54.S1, R54.S2, R55.1, R55.S1, R55.S2, R56.1, R56.S1, R56.S2, R57.1, R57.S1, R57.S2, R58.1, R58.S1, R58.S2, R59.1, R59.S1, R59.S2, R60.1, R60.S1, R60.S2, R61.1, R61.S1, R61.S2, R62.1, R62.S1, R62.S2, R63.1, R63.S1, R63.S2, R64.1, R64.S1, R64.S2, U2.12, U2.15, U3.12, U3.15, U4.12, U4.15; no longer CONN2.5, CONN3.6
- net MUX_COMMON_1: now also CONN1.1, U1.1; no longer CONN1.4, CONN2.7, CONN3.4, R17.2
- net MUX_COMMON_2: now also CONN1.2, U2.1; no longer CONN1.3, CONN2.8, CONN3.3, R18.2
- net MUX_COMMON_3: now also CONN1.3, U3.1; no longer CONN1.2, CONN2.9, CONN3.2, R19.2
- net MUX_COMMON_4: now also CONN1.4, U4.1; no longer CONN1.1, CONN2.10, CONN3.1, R20.2
- net MUX_S0: now also U2.10, U3.10, U4.10; no longer CONN2.3, CONN3.8
- net MUX_S1: now also U2.11, U3.11, U4.11; no longer CONN2.4, CONN3.7
- net MUX_S2: now also U2.14, U3.14, U4.14; no longer CONN2.2, CONN3.9
- net MUX_S3: now also U2.13, U3.13, U4.13; no longer CONN2.1, CONN3.10
Routing:
- net +3V3: track 642.2 -> 2328.8 mm, vias 2 -> 0
- net MUX_S3: track 79.6 -> 423.3 mm, vias 2 -> 5
- net MUX_S2: track 81.6 -> 420.6 mm, vias 2 -> 5
- net MUX_COMMON_1: track 68.4 -> 403.9 mm, vias 0 -> 2
- net MUX_S0: track 85.1 -> 406.1 mm, vias 2 -> 5
- net MUX_S1: track 82.2 -> 397.9 mm, vias 2 -> 5
- net MUX_COMMON_2: track 66.9 -> 285.5 mm, vias 0 -> 2
- net MUX_COMMON_3: track 72.1 -> 167.6 mm, vias 0 -> 2
- net POT17: track 0.00 -> 66.0 mm
- net POT49: track 0.00 -> 66.0 mm
- net POT33: track 0.00 -> 66.0 mm
- net POT61: track 0.00 -> 64.0 mm
- net POT45: track 0.00 -> 64.0 mm
- net POT29: track 0.00 -> 64.0 mm
- net POT20: track 0.00 -> 62.1 mm
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Other:
- board size 135.2 x 99.8 mm -> 449.6 x 100.3 mm
- board text removed: "IN"
- board text removed: "OUT"
