File: bin/sch/dubfocus/Pots/Pots.sch (EAGLE design)
At the start: 27 parts, among them U1 MC14067BDWR2G-SO24W

Commit message: targets: update schematics for dubfocus
Parts:
- removed CONN2, CONN3: PINHD-1X10-FFC-1MM-Z, igor_lbr:PINHD-1X10-FFC-1MM-Z
- added C4, C5, C6: 100n, igor_lbr:CAPACITOR-0805
- added R21, R22, R23, R24, R25, R26, R27, R28, R29, R30, R31, R32, R33, R34, R35, R36, R37, R38, R39, R40, R41, R42, R43, R44, R45, R46, R47, R48, R49, R50, R51, R52, R53, R54, R55, R56, R57, R58, R59, R60, R61, R62, R63, R64: 10k, igor_lbr:PTV09A-4025F-B103
- added U2, U3, U4: MC14067BDWR2G-SO24W, igor_lbr:MC14067BDWR2G-SO24W
- R17, R18, R19, R20: value 0 -> 10k; device igor_lbr:RESISTOR-0805 -> igor_lbr:PTV09A-4025F-B103
Connections:
- removed net MUX_COMMON: R17.1, R18.1, R19.1, R20.1, U1.Z
- new net POT17: R17-POT.2, U2.Y10
- new net POT18: R18-POT.2, U2.Y11
- new net POT19: R19-POT.2, U2.Y12
- new net POT20: R20-POT.2, U2.Y13
- new net POT21: R21-POT.2, U2.Y8
- new net POT22: R22-POT.2, U2.Y9
- new net POT23: R23-POT.2, U2.Y14
- new net POT24: R24-POT.2, U2.Y15
- new net POT25: R25-POT.2, U2.Y7
- new net POT26: R26-POT.2, U2.Y6
- new net POT27: R27-POT.2, U2.Y1
- new net POT28: R28-POT.2, U2.Y0
- new net POT29: R29-POT.2, U2.Y5
- new net POT30: R30-POT.2, U2.Y4
- new net POT31: R31-POT.2, U2.Y3
- new net POT32: R32-POT.2, U2.Y2
- new net POT33: R33-POT.2, U3.Y10
- new net POT34: R34-POT.2, U3.Y11
- new net POT35: R35-POT.2, U3.Y12
- new net POT36: R36-POT.2, U3.Y13
- new net POT37: R37-POT.2, U3.Y8
- new net POT38: R38-POT.2, U3.Y9
- new net POT39: R39-POT.2, U3.Y14
- new net POT40: R40-POT.2, U3.Y15
- new net POT41: R41-POT.2, U3.Y7
- new net POT42: R42-POT.2, U3.Y6
- new net POT43: R43-POT.2, U3.Y1
- new net POT44: R44-POT.2, U3.Y0
- new net POT45: R45-POT.2, U3.Y5
- new net POT46: R46-POT.2, U3.Y4
- new net POT47: R47-POT.2, U3.Y3
- new net POT48: R48-POT.2, U3.Y2
- new net POT49: R49-POT.2, U4.Y10
- new net POT50: R50-POT.2, U4.Y11
- new net POT51: R51-POT.2, U4.Y12
- new net POT52: R52-POT.2, U4.Y13
- new net POT53: R53-POT.2, U4.Y8
- new net POT54: R54-POT.2, U4.Y9
- new net POT55: R55-POT.2, U4.Y14
- new net POT56: R56-POT.2, U4.Y15
- new net POT57: R57-POT.2, U4.Y7
- new net POT58: R58-POT.2, U4.Y6
- new net POT59: R59-POT.2, U4.Y1
- new net POT60: R60-POT.2, U4.Y0
- new net POT61: R61-POT.2, U4.Y5
- new net POT62: R62-POT.2, U4.Y4
- new net POT63: R63-POT.2, U4.Y3
- new net POT64: R64-POT.2, U4.Y2
- net +3V3: now also C4.2, C5.2, C6.2, R17-POT.3, R18-POT.3, R19-POT.3, R20-POT.3, R21-POT.3, R22-POT.3, R23-POT.3, R24-POT.3, R25-POT.3, R26-POT.3, R27-POT.3, R28-POT.3, R29-POT.3, R30-POT.3, R31-POT.3, R32-POT.3, R33-POT.3, R34-POT.3, R35-POT.3, R36-POT.3, R37-POT.3, R38-POT.3, R39-POT.3, R40-POT.3, R41-POT.3, R42-POT.3, R43-POT.3, R44-POT.3, R45-POT.3, R46-POT.3, R47-POT.3, R48-POT.3, R49-POT.3, R50-POT.3, R51-POT.3, R52-POT.3, R53-POT.3, R54-POT.3, R55-POT.3, R56-POT.3, R57-POT.3, R58-POT.3, R59-POT.3, R60-POT.3, R61-POT.3, R62-POT.3, R63-POT.3, R64-POT.3, U2.VCC, U3.VCC, U4.VCC; no longer CONN2.6, CONN3.5
- net GND: now also C4.1, C5.1, C6.1, R17-POT.1, R17-S1.S, R17-S2.S, R18-POT.1, R18-S1.S, R18-S2.S, R19-POT.1, R19-S1.S, R19-S2.S, R20-POT.1, R20-S1.S, R20-S2.S, R21-POT.1, R21-S1.S, R21-S2.S, R22-POT.1, R22-S1.S, R22-S2.S, R23-POT.1, R23-S1.S, R23-S2.S, R24-POT.1, R24-S1.S, R24-S2.S, R25-POT.1, R25-S1.S, R25-S2.S, R26-POT.1, R26-S1.S, R26-S2.S, R27-POT.1, R27-S1.S, R27-S2.S, R28-POT.1, R28-S1.S, R28-S2.S, R29-POT.1, R29-S1.S, R29-S2.S, R30-POT.1, R30-S1.S, R30-S2.S, R31-POT.1, R31-S1.S, R31-S2.S, R32-POT.1, R32-S1.S, R32-S2.S, R33-POT.1, R33-S1.S, R33-S2.S, R34-POT.1, R34-S1.S, R34-S2.S, R35-POT.1, R35-S1.S, R35-S2.S, R36-POT.1, R36-S1.S, R36-S2.S, R37-POT.1, R37-S1.S, R37-S2.S, R38-POT.1, R38-S1.S, R38-S2.S, R39-POT.1, R39-S1.S, R39-S2.S, R40-POT.1, R40-S1.S, R40-S2.S, R41-POT.1, R41-S1.S, R41-S2.S, R42-POT.1, R42-S1.S, R42-S2.S, R43-POT.1, R43-S1.S, R43-S2.S, R44-POT.1, R44-S1.S, R44-S2.S, R45-POT.1, R45-S1.S, R45-S2.S, R46-POT.1, R46-S1.S, R46-S2.S, R47-POT.1, R47-S1.S, R47-S2.S, R48-POT.1, R48-S1.S, R48-S2.S, R49-POT.1, R49-S1.S, R49-S2.S, R50-POT.1, R50-S1.S, R50-S2.S, R51-POT.1, R51-S1.S, R51-S2.S, R52-POT.1, R52-S1.S, R52-S2.S, R53-POT.1, R53-S1.S, R53-S2.S, R54-POT.1, R54-S1.S, R54-S2.S, R55-POT.1, R55-S1.S, R55-S2.S, R56-POT.1, R56-S1.S, R56-S2.S, R57-POT.1, R57-S1.S, R57-S2.S, R58-POT.1, R58-S1.S, R58-S2.S, R59-POT.1, R59-S1.S, R59-S2.S, R60-POT.1, R60-S1.S, R60-S2.S, R61-POT.1, R61-S1.S, R61-S2.S, R62-POT.1, R62-S1.S, R62-S2.S, R63-POT.1, R63-S1.S, R63-S2.S, R64-POT.1, R64-S1.S, R64-S2.S, U2.!E, U2.GND, U3.!E, U3.GND, U4.!E, U4.GND; no longer CONN2.5, CONN3.6
- net MUX_COMMON_1: now also CONN1.1, U1.Z; no longer CONN1.4, CONN2.7, CONN3.4, R17.2
- net MUX_COMMON_2: now also CONN1.2, U2.Z; no longer CONN1.3, CONN2.8, CONN3.3, R18.2
- net MUX_COMMON_3: now also CONN1.3, U3.Z; no longer CONN1.2, CONN2.9, CONN3.2, R19.2
- net MUX_COMMON_4: now also CONN1.4, U4.Z; no longer CONN1.1, CONN2.10, CONN3.1, R20.2
- net MUX_S0: now also U2.S0, U3.S0, U4.S0; no longer CONN2.3, CONN3.8
- net MUX_S1: now also U2.S1, U3.S1, U4.S1; no longer CONN2.4, CONN3.7
- net MUX_S2: now also U2.S2, U3.S2, U4.S2; no longer CONN2.2, CONN3.9
- net MUX_S3: now also U2.S3, U3.S3, U4.S3; no longer CONN2.1, CONN3.10
Other:
- note removed: "Note: same-sided flat cables should be used, such as Molex 15267-0257 Board closest to the MBO should have 0ohm resistor mounted on R17. Second board: R18 Third and fourth board should follow the same pattern. For unused boards do not mount resistor."
- moved on the sheet: C1, C2, C3, CONN1, R1-POT, R1-S1, R1-S2, R10-POT, R10-S1, R10-S2, R11-POT, R11-S1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
