File: bin/sch/opendeck/v2.1.0/OpenDeck-r2.1.0.brd (EAGLE design)
At the start: 99.8 x 99.8 mm, 114 parts, among them U1 STM32F405RGT6-10X10, U2 6N137-SMD, U3 MAX7219, U4 74HC138-SO, U5 MC14067BDWR2G-SO24W, U6 MC14067BDWR2G-SO24W, U7 74125-TSSOP, Y1 12MHz

Commit message: sch: fix signal names for max7219 in opendeck 2.1
Connections:
- net DEC_DO_A0 renamed MAX7219_DIN
- net DEC_DO_A1 renamed MAX7219_LOAD
- net DEC_DO_A2 renamed MAX7219_CLK
Changed lines of the file:
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@@
 <signal name="S$121">
 </signal>
-<signal name="DEC_DO_A0">
+<signal name="MAX7219_DIN">
 <contactref element="U1" pad="16"/>
 <wire x1="90.969" y1="89.094" x2="91.38" y2="89.094" width="0.2032" layer="1"/>
@@
 <wire x1="76.708" y1="4.064" x2="76.708" y2="13.716" width="0.2032" layer="16"/>
 </signal>
-<signal name="DEC_DO_A1">
+<signal name="MAX7219_LOAD">
 <contactref element="U1" pad="15"/>
 <via x="93.218" y="90.932" extent="1-16" drill="0.4"/>
@@
 <contactref element="U1" pad="17"/>
 </signal>
-<signal name="DEC_DO_A2">
+<signal name="MAX7219_CLK">
 <contactref element="U1" pad="14"/>
 <wire x1="90.969" y1="88.094" x2="92.158" y2="88.094" width="0.2032" layer="1"/>
