File: bin/sch/opendeck/v2.1.0/OpenDeck-r2.1.0.sch (EAGLE design)
At the start: 114 parts, among them U1 STM32F405RGT6-10X10, U2 6N137-SMD, U3 MAX7219, U4 74HC138-SO, U5 MC14067BDWR2G-SO24W, U6 MC14067BDWR2G-SO24W, U7 74125-TSSOP, Y1 12MHz

Commit message: sch: fix signal names for max7219 in opendeck 2.1
Connections:
- net DEC_DO_A0 renamed MAX7219_DIN
- net DEC_DO_A1 renamed MAX7219_LOAD
- net DEC_DO_A2 renamed MAX7219_CLK
Changed lines of the file:
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@@
 <attribute name="LCSC" x="147.32" y="101.6" size="1.778" layer="96" rot="R180" display="off"/>
 </instance>
-<instance part="GND35" gate="1" x="127" y="91.44" smashed="yes" rot="R270">
-<attribute name="VALUE" x="124.46" y="93.98" size="1.778" layer="96" font="vector" rot="R270"/>
+<instance part="GND35" gate="1" x="124.46" y="91.44" smashed="yes" rot="R270">
+<attribute name="VALUE" x="121.92" y="93.98" size="1.778" layer="96" font="vector" rot="R270"/>
 </instance>
 <instance part="C19" gate="C" x="124.46" y="195.58">
@@
 <instance part="U7" gate="-GND" x="154.94" y="91.44" rot="R90"/>
 <instance part="U7" gate="-VCC" x="154.94" y="93.98" rot="R90"/>
-<instance part="GND36" gate="1" x="127" y="83.82" smashed="yes" rot="R270">
-<attribute name="VALUE" x="124.46" y="86.36" size="1.778" layer="96" font="vector" rot="R270"/>
+<instance part="GND36" gate="1" x="124.46" y="83.82" smashed="yes" rot="R270">
+<attribute name="VALUE" x="121.92" y="86.36" size="1.778" layer="96" font="vector" rot="R270"/>
 </instance>
-<instance part="GND37" gate="1" x="127" y="78.74" smashed="yes" rot="R270">
-<attribute name="VALUE" x="124.46" y="81.28" size="1.778" layer="96" font="vector" rot="R270"/>
+<instance part="GND37" gate="1" x="124.46" y="78.74" smashed="yes" rot="R270">
+<attribute name="VALUE" x="121.92" y="81.28" size="1.778" layer="96" font="vector" rot="R270"/>
 </instance>
-<instance part="GND38" gate="1" x="127" y="73.66" smashed="yes" rot="R270">
-<attribute name="VALUE" x="124.46" y="76.2" size="1.778" layer="96" font="vector" rot="R270"/>
+<instance part="GND38" gate="1" x="124.46" y="73.66" smashed="yes" rot="R270">
+<attribute name="VALUE" x="121.92" y="76.2" size="1.778" layer="96" font="vector" rot="R270"/>
 </instance>
 <instance part="GND44" gate="1" x="185.42" y="99.06" smashed="yes" rot="R180">
@@
 <segment>
 <pinref part="GND35" gate="1" pin="GND"/>
-<wire x1="129.54" y1="91.44" x2="149.86" y2="91.44" width="0.1524" layer="91"/>
+<wire x1="127" y1="91.44" x2="149.86" y2="91.44" width="0.1524" layer="91"/>
 <pinref part="U7" gate="-GND" pin="VEE"/>
 </segment>
@@
 <pinref part="U7" gate="-GATES" pin="1!(OE)"/>
 <pinref part="GND36" gate="1" pin="GND"/>
-<wire x1="129.54" y1="83.82" x2="144.78" y2="83.82" width="0.1524" layer="91"/>
+<wire x1="127" y1="83.82" x2="144.78" y2="83.82" width="0.1524" layer="91"/>
 </segment>
 <segment>
 <pinref part="U7" gate="-GATES" pin="2!(OE)"/>
 <pinref part="GND37" gate="1" pin="GND"/>
-<wire x1="129.54" y1="78.74" x2="144.78" y2="78.74" width="0.1524" layer="91"/>
+<wire x1="127" y1="78.74" x2="144.78" y2="78.74" width="0.1524" layer="91"/>
 </segment>
 <segment>
 <pinref part="U7" gate="-GATES" pin="3!(OE)"/>
 <pinref part="GND38" gate="1" pin="GND"/>
-<wire x1="129.54" y1="73.66" x2="144.78" y2="73.66" width="0.1524" layer="91"/>
+<wire x1="127" y1="73.66" x2="144.78" y2="73.66" width="0.1524" layer="91"/>
 </segment>
 <segment>
@@
 </segment>
 </net>
-<net name="DEC_DO_A0" class="0">
+<net name="MAX7219_DIN" class="0">
 <segment>
 <label x="142.24" y="86.36" size="1.27" layer="95" font="vector" rot="R180" xref="yes"/>
@@
 </segment>
 </net>
-<net name="DEC_DO_A1" class="0">
+<net name="MAX7219_LOAD" class="0">
 <segment>
 <label x="142.24" y="81.28" size="1.27" layer="95" font="vector" rot="R180" xref="yes"/>
@@
 </segment>
 </net>
-<net name="DEC_DO_A2" class="0">
+<net name="MAX7219_CLK" class="0">
 <segment>
 <pinref part="U1" gate="G$1" pin="PA0"/>
