File: bin/sch/opendeck/v3.1.x/Analog_Multiplexer.kicad_sch (KiCad schematic)
At the start: 4 parts, among them U1 74HC4067

Commit message: sch: update opendeck 3.1 schematics
replace SOIC-24 package for the multiplexers with TSSOP-24
Parts:
- U1: footprint Package_SO:SOIC-24W_7.5x15.4mm_P1.27mm -> Package_SO:TSSOP-24_4.4x7.8mm_P0.65mm; LCSC C496123 -> C179326
