File: bin/sch/dubfocus/16t/ButtonsLEDs/ButtonsLEDs.kicad_pcb (KiCad board)
At the start: 2 copper layers, 390 x 37 mm, 100 parts, among them U1 74HC165, U2 74HC165, U3 74HC165, U4 74HC165, U5 MAX7219, U6 74HCT125, U9 74HCT125

Commit message: sch/dubfocus16t: misc updates
Parts:
- moved H5 0.68 mm to (516.5, 185.0)
- moved H7 0.65 mm to (516.5, 160.0)
- moved H4 0.47 mm to (166.5, 160.0)
- moved H8 0.32 mm to (166.5, 185.0)
Routing:
- net /Buttons 4/BUTTON4: track 34.6 -> 38.2 mm
Other:
- outline, holes or cut-outs redrawn
Changed lines of the file:
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@@
 	(footprint "MountingHole:MountingHole_2.5mm_Pad"
 		(layer "F.Cu")
-		(at 166.2 185.1)
+		(at 166.5 185)
 		(descr "Mounting Hole 2.5mm, generated by kicad-footprint-generator mountinghole.py")
 		(tags "mountinghole")
@@
 	(footprint "MountingHole:MountingHole_2.5mm_Pad"
 		(layer "F.Cu")
-		(at 166.9 160.25)
+		(at 166.5 160)
 		(descr "Mounting Hole 2.5mm, generated by kicad-footprint-generator mountinghole.py")
 		(tags "mountinghole")
@@
 	(footprint "MountingHole:MountingHole_2.5mm_Pad"
 		(layer "F.Cu")
-		(at 516.15 160.55)
+		(at 516.5 160)
 		(descr "Mounting Hole 2.5mm, generated by kicad-footprint-generator mountinghole.py")
 		(tags "mountinghole")
@@
 	(footprint "MountingHole:MountingHole_2.5mm_Pad"
 		(layer "F.Cu")
-		(at 515.95 185.4)
+		(at 516.5 185)
 		(descr "Mounting Hole 2.5mm, generated by kicad-footprint-generator mountinghole.py")
 		(tags "mountinghole")
@@
 		(layer "B.SilkS")
 	)
-	(gr_line
-		(start 146.5 176.55)
-		(end 146.5 191.5)
-		(stroke
-			(width 0.1)
-			(type default)
-		)
-		(layer "Edge.Cuts")
-	)
-	(gr_line
+	(gr_rect
 		(start 146.5 154.5)
-		(end 146.5 168.4)
-		(stroke
-			(width 0.1)
-			(type default)
-		)
-		(layer "Edge.Cuts")
-	)
-	(gr_line
-		(start 536.5 154.5)
-		(end 146.5 154.5)
-		(stroke
-			(width 0.1)
-			(type default)
-		)
-		(layer "Edge.Cuts")
-	)
-	(gr_line
-		(start 532 176.55)
-		(end 536.5 176.55)
-		(stroke
-			(width 0.1)
-			(type solid)
-		)
-		(layer "Edge.Cuts")
-	)
-	(gr_line
-		(start 532 176.55)
-		(end 532 168.4)
-		(stroke
-			(width 0.1)
-			(type default)
-		)
-		(layer "Edge.Cuts")
-	)
-	(gr_line
-		(start 150.95 176.55)
-		(end 146.5 176.55)
-		(stroke
-			(width 0.1)
-			(type solid)
-		)
-		(layer "Edge.Cuts")
-	)
-	(gr_line
-		(start 536.5 168.4)
-		(end 536.5 154.5)
-		(stroke
-			(width 0.1)
-			(type default)
-		)
-		(layer "Edge.Cuts")
-	)
-	(gr_line
-		(start 146.5 191.5)
 		(end 536.5 191.5)
 		(stroke
@@
 			(type default)
 		)
-		(layer "Edge.Cuts")
-	)
-	(gr_line
-		(start 150.95 168.4)
-		(end 150.95 176.55)
-		(stroke
-			(width 0.1)
-			(type default)
-		)
-		(layer "Edge.Cuts")
-	)
-	(gr_line
-		(start 536.5 191.5)
-		(end 536.5 176.55)
-		(stroke
-			(width 0.1)
-			(type default)
-		)
-		(layer "Edge.Cuts")
-	)
-	(gr_line
-		(start 150.95 168.4)
-		(end 146.5 168.4)
-		(stroke
-			(width 0.1)
-			(type default)
-		)
-		(layer "Edge.Cuts")
-	)
-	(gr_line
-		(start 532 168.4)
-		(end 536.5 168.4)
-		(stroke
-			(width 0.1)
-			(type solid)
-		)
+		(fill no)
 		(layer "Edge.Cuts")
 	)
@@
 	)
 	(segment
+		(start 523 157.325)
+		(end 525.325 157.325)
+		(width 0.2)
+		(layer "B.Cu")
+		(net 35)
+	)
+	(segment
+		(start 509.805 170.325)
+		(end 509.805 159.145)
+		(width 0.2)
+		(layer "B.Cu")
+		(net 35)
+	)
+	(segment
 		(start 525.75 157.75)
 		(end 532.25 157.75)
@@
 	)
 	(segment
-		(start 525.325 157.325)
-		(end 525.75 157.75)
+		(start 509.805 159.145)
+		(end 512.525 156.425)
 		(width 0.2)
 		(layer "B.Cu")
@@
 	)
 	(segment
-		(start 509.805 159.145)
-		(end 511.625 157.325)
+		(start 512.525 156.425)
+		(end 524.425 156.425)
 		(width 0.2)
 		(layer "B.Cu")
@@
 	)
 	(segment
-		(start 509.805 170.325)
-		(end 509.805 159.145)
+		(start 525.325 157.325)
+		(end 525.75 157.75)
 		(width 0.2)
 		(layer "B.Cu")
@@
 	)
 	(segment
-		(start 511.625 157.325)
-		(end 525.325 157.325)
+		(start 524.425 156.425)
+		(end 525.75 157.75)
 		(width 0.2)
 		(layer "B.Cu")
