File: bin/sch/dubfocus/16t/MBO/MBO.kicad_pcb (KiCad board)
At the start: 2 copper layers, 390 x 78.2 mm, 45 parts, among them U2 MCP1825S, U3 MC14067BDWR2G-SO24W, U5 STM32F405RGTx, Y1 8MHz

Commit message: sch/dubfocus16t: misc updates
Parts:
- added H1: MountingHole_Pad, MountingHole:MountingHole_2.5mm_Pad, F.Cu at (166.5, 158.0)
- added H10: MountingHole_Pad, MountingHole:MountingHole_2.5mm_Pad, F.Cu at (366.5, 209.2)
- added H11: MountingHole_Pad, MountingHole:MountingHole_2.5mm_Pad, F.Cu at (416.5, 158.0)
- added H12: MountingHole_Pad, MountingHole:MountingHole_2.5mm_Pad, F.Cu at (416.5, 229.2)
- added H13: MountingHole_Pad, MountingHole:MountingHole_2.5mm_Pad, F.Cu at (466.5, 158.0)
- added H14: MountingHole_Pad, MountingHole:MountingHole_2.5mm_Pad, F.Cu at (466.5, 229.2)
- added H15: MountingHole_Pad, MountingHole:MountingHole_2.5mm_Pad, F.Cu at (516.5, 158.0)
- added H16: MountingHole_Pad, MountingHole:MountingHole_2.5mm_Pad, F.Cu at (516.5, 229.2)
- added H2: MountingHole_Pad, MountingHole:MountingHole_2.5mm_Pad, F.Cu at (166.5, 229.2)
- added H3: MountingHole_Pad, MountingHole:MountingHole_2.5mm_Pad, F.Cu at (216.5, 158.0)
- added H4: MountingHole_Pad, MountingHole:MountingHole_2.5mm_Pad, F.Cu at (216.5, 229.2)
- added H5: MountingHole_Pad, MountingHole:MountingHole_2.5mm_Pad, F.Cu at (266.5, 158.0)
- added H6: MountingHole_Pad, MountingHole:MountingHole_2.5mm_Pad, F.Cu at (266.5, 229.2)
- added H7: MountingHole_Pad, MountingHole:MountingHole_2.5mm_Pad, F.Cu at (316.5, 178.0)
- added H8: MountingHole_Pad, MountingHole:MountingHole_2.5mm_Pad, F.Cu at (316.5, 209.2)
- added H9: MountingHole_Pad, MountingHole:MountingHole_2.5mm_Pad, F.Cu at (366.5, 178.0)
- moved CONN4 2.38 mm to (517.1, 203.4)
- moved R3 1.43 mm to (516.8, 173.4)
- moved U2 1.33 mm to (517.3, 167.0)
- moved FB1 1.10 mm to (512.5, 164.1)
- moved C11 1.04 mm to (513.1, 170.2)
Routing:
- net +3.3VADC: track 528.2 -> 534.7 mm
- net +3V3: track 109.3 -> 112.5 mm
- net /NRST: track 39.7 -> 42.2 mm
- net /SWDCLK: track 9.62 -> 11.8 mm
- net /SWDIO: track 19.9 -> 22.1 mm
- net /MCU/BTLDR_BUTTON: track 215.8 -> 215.3 mm
- net GND: vias 44 -> 45
