File: bin/sch/dubfocus/16t/MBO/MBO.kicad_sch (KiCad schematic)
At the start: 0 parts

Commit message: sch/dubfocus16t: misc updates
Parts:
- added H1, H10, H11, H12, H13, H14, H15, H16, H2, H3, H4, H5, H6, H7, H8, H9: MountingHole_Pad, MountingHole:MountingHole_2.5mm_Pad, symbol Mechanical:MountingHole_Pad
Connections:
- new net GNDA: H1.1, H10.1, H11.1, H12.1, H13.1, H14.1, H15.1, H16.1, H2.1, H3.1, H4.1, H5.1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
