File: bin/sch/dubfocus/16t/Pots/Pots.kicad_pcb (KiCad board)
At the start: 2 copper layers, 390 x 93 mm, 93 parts, among them U1 MC14067BDWR2G-SO24W, U2 MC14067BDWR2G-SO24W, U3 MC14067BDWR2G-SO24W, U4 MC14067BDWR2G-SO24W

Commit message: sch/dubfocus16t: misc updates
Other:
- outline, holes or cut-outs redrawn
Changed lines of the file:
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@@
 		(layer "B.SilkS")
 	)
-	(gr_line
-		(start 536.505 179.5)
+	(gr_rect
+		(start 146.5 154.5)
 		(end 536.5 247.5)
 		(stroke
@@
 			(type default)
 		)
+		(fill no)
 		(layer "Edge.Cuts")
 	)
-	(gr_line
-		(start 146.5 171.5)
-		(end 146.5 154.5)
-		(stroke
-			(width 0.1)
-			(type default)
-		)
-		(layer "Edge.Cuts")
-	)
-	(gr_line
-		(start 152.5 171.5)
-		(end 146.5 171.5)
-		(stroke
-			(width 0.1)
-			(type default)
-		)
-		(layer "Edge.Cuts")
-	)
-	(gr_line
-		(start 536.5 171.5)
-		(end 530.505 171.5)
-		(stroke
-			(width 0.1)
-			(type default)
-		)
-		(layer "Edge.Cuts")
-	)
-	(gr_line
-		(start 146.5 247.5)
-		(end 146.5 179.5)
-		(stroke
-			(width 0.1)
-			(type default)
-		)
-		(layer "Edge.Cuts")
-	)
-	(gr_line
-		(start 146.5 179.5)
-		(end 152.5 179.5)
-		(stroke
-			(width 0.1)
-			(type default)
-		)
-		(layer "Edge.Cuts")
-	)
-	(gr_line
-		(start 536.5 247.5)
-		(end 146.5 247.5)
-		(stroke
-			(width 0.1)
-			(type default)
-		)
-		(layer "Edge.Cuts")
-	)
-	(gr_line
-		(start 152.5 179.5)
-		(end 152.5 171.5)
-		(stroke
-			(width 0.1)
-			(type default)
-		)
-		(layer "Edge.Cuts")
-	)
-	(gr_line
-		(start 530.505 171.5)
-		(end 530.505 179.5)
-		(stroke
-			(width 0.1)
-			(type default)
-		)
-		(layer "Edge.Cuts")
-	)
-	(gr_line
-		(start 536.5 154.5)
-		(end 536.5 171.5)
-		(stroke
-			(width 0.1)
-			(type default)
-		)
-		(layer "Edge.Cuts")
-	)
-	(gr_line
-		(start 530.505 179.5)
-		(end 536.5 179.5)
-		(stroke
-			(width 0.1)
-			(type default)
-		)
-		(layer "Edge.Cuts")
-	)
-	(gr_line
-		(start 146.5 154.5)
-		(end 536.5 154.5)
-		(stroke
-			(width 0.1)
-			(type default)
-		)
-		(layer "Edge.Cuts")
-	)
